File: hw/stm32-pillbus/pillbus.kicad_sch (KiCad schematic)
At the start: 9 parts, among them J1 LEDs DI, J2 LEDs DI, J3 LEDs DI, J4 LEDs DI, J5 LEDs DO, J6 LEDs DO, J7 LEDs DO, J8 LEDs DO

Commit message: stm32pill schema
Other:
- added sheet stm32pill (stm32pill.kicad_sch)
- added sheet stm32pill1 (stm32pill.kicad_sch)
- added sheet stm32pill2 (stm32pill.kicad_sch)
- added sheet stm32pill3 (stm32pill.kicad_sch)
- added sheet stm32pill4 (stm32pill.kicad_sch)
- moved on the sheet: R1
Changed lines of the file:
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@@
 	(wire
 		(pts
-			(xy 26.67 24.13) (xy 33.02 24.13)
+			(xy 156.21 146.05) (xy 162.56 146.05)
 		)
 		(stroke
@@
 	(symbol
 		(lib_id "Device:R")
-		(at 26.67 27.94 0)
+		(at 156.21 149.86 0)
 		(unit 1)
 		(exclude_from_sim no)
@@
 		(fields_autoplaced yes)
 		(property "Reference" "R1"
-			(at 29.21 26.6699 0)
+			(at 158.75 148.5899 0)
 			(effects
 				(font
@@
 		)
 		(property "Value" "R"
-			(at 29.21 29.2099 0)
+			(at 158.75 151.1299 0)
 			(effects
 				(font
@@
 		)
 		(property "Footprint" ""
-			(at 24.892 27.94 90)
+			(at 154.432 149.86 90)
 			(effects
 				(font
@@
 		)
 		(property "Datasheet" "~"
-			(at 26.67 27.94 0)
+			(at 156.21 149.86 0)
 			(effects
 				(font
@@
 		)
 		(property "Description" "Resistor"
-			(at 26.67 27.94 0)
+			(at 156.21 149.86 0)
 			(effects
 				(font
@@
 	(symbol
 		(lib_id "power:GND")
-		(at 26.67 31.75 0)
+		(at 156.21 153.67 0)
 		(unit 1)
 		(exclude_from_sim no)
@@
 		(fields_autoplaced yes)
 		(property "Reference" "#PWR09"
-			(at 26.67 38.1 0)
+			(at 156.21 160.02 0)
 			(effects
 				(font
@@
 		)
 		(property "Value" "GND"
-			(at 26.67 36.83 0)
+			(at 156.21 158.75 0)
 			(effects
 				(font
@@
 		)
 		(property "Footprint" ""
-			(at 26.67 31.75 0)
+			(at 156.21 153.67 0)
 			(effects
 				(font
@@
 		)
 		(property "Datasheet" ""
-			(at 26.67 31.75 0)
+			(at 156.21 153.67 0)
 			(effects
 				(font
@@
 		)
 		(property "Description" "Power symbol creates a global label with name \"GND\" , ground"
-			(at 26.67 31.75 0)
+			(at 156.21 153.67 0)
 			(effects
 				(font
@@
 	(symbol
 		(lib_id "power:GND")
-		(at 33.02 24.13 0)
+		(at 162.56 146.05 0)
 		(unit 1)
 		(exclude_from_sim no)
@@
 		(fields_autoplaced yes)
 		(property "Reference" "#PWR08"
-			(at 33.02 30.48 0)
+			(at 162.56 152.4 0)
 			(effects
 				(font
@@
 		)
 		(property "Value" "GND"
-			(at 33.02 29.21 0)
+			(at 162.56 151.13 0)
 			(effects
 				(font
@@
 		)
 		(property "Footprint" ""
-			(at 33.02 24.13 0)
+			(at 162.56 146.05 0)
 			(effects
 				(font
@@
 		)
 		(property "Datasheet" ""
-			(at 33.02 24.13 0)
+			(at 162.56 146.05 0)
 			(effects
 				(font
@@
 		)
 		(property "Description" "Power symbol creates a global label with name \"GND\" , ground"
-			(at 33.02 24.13 0)
+			(at 162.56 146.05 0)
 			(effects
 				(font
@@
 	)
 	(sheet
-		(at 196.85 138.43)
-		(size 74.93 8.89)
+		(at 213.36 24.13)
+		(size 43.18 59.69)
 		(fields_autoplaced yes)
 		(stroke
@@
 			(color 0 0 0 0.0000)
 		)
+		(property "Sheetname" "stm32pill3"
+			(at 213.36 23.4184 0)
+			(effects
+				(font
+					(size 1.27 1.27)
+				)
+				(justify left bottom)
+			)
+		)
+		(property "Sheetfile" "stm32pill.kicad_sch"
+			(at 213.36 84.4046 0)
+			(effects
+				(font
+					(size 1.27 1.27)
+				)
+				(justify left top)
+			)
+		)
+		(instances
+			(project "pillbus"
+				(path "/eae9d418-f407-4ce6-ae70-138b36f2a986"
+					(page "9")
+				)
+			)
+		)
+	)
+	(sheet
+		(at 196.85 138.43)
+		(size 74.93 8.89)
+		(fields_autoplaced yes)
+		(stroke
+			(width 0.1524)
+			(type solid)
+		)
+		(fill
+			(color 0 0 0 0.0000)
+		)
 		(property "Sheetname" "leds1"
 			(at 196.85 137.7184 0)
@@
 				(path "/eae9d418-f407-4ce6-ae70-138b36f2a986"
 					(page "3")
+				)
+			)
+		)
+	)
+	(sheet
+		(at 83.82 22.86)
+		(size 43.18 59.69)
+		(fields_autoplaced yes)
+		(stroke
+			(width 0.1524)
+			(type solid)
+		)
+		(fill
+			(color 0 0 0 0.0000)
+		)
+		(property "Sheetname" "stm32pill1"
+			(at 83.82 22.1484 0)
+			(effects
+				(font
+					(size 1.27 1.27)
+				)
+				(justify left bottom)
+			)
+		)
+		(property "Sheetfile" "stm32pill.kicad_sch"
+			(at 83.82 83.1346 0)
+			(effects
+				(font
+					(size 1.27 1.27)
+				)
+				(justify left top)
+			)
+		)
+		(instances
+			(project "pillbus"
+				(path "/eae9d418-f407-4ce6-ae70-138b36f2a986"
+					(page "7")
 				)
 			)
@@
 	)
 	(sheet
-		(at 196.85 121.92)
-		(size 74.93 8.89)
+		(at 83.82 109.22)
+		(size 43.18 59.69)
 		(fields_autoplaced yes)
 		(stroke
@@
 			(color 0 0 0 0.0000)
 		)
+		(property "Sheetname" "stm32pill4"
+			(at 83.82 108.5084 0)
+			(effects
+				(font
+					(size 1.27 1.27)
+				)
+				(justify left bottom)
+			)
+		)
+		(property "Sheetfile" "stm32pill.kicad_sch"
+			(at 83.82 169.4946 0)
+			(effects
+				(font
+					(size 1.27 1.27)
+				)
+				(justify left top)
+			)
+		)
+		(instances
+			(project "pillbus"
+				(path "/eae9d418-f407-4ce6-ae70-138b36f2a986"
+					(page "10")
+				)
+			)
+		)
+	)
+	(sheet
+		(at 147.32 22.86)
+		(size 43.18 59.69)
+		(fields_autoplaced yes)
+		(stroke
+			(width 0.1524)
+			(type solid)
+		)
+		(fill
+			(color 0 0 0 0.0000)
+		)
+		(property "Sheetname" "stm32pill2"
+			(at 147.32 22.1484 0)
+			(effects
+				(font
+					(size 1.27 1.27)
+				)
+				(justify left bottom)
+			)
+		)
+		(property "Sheetfile" "stm32pill.kicad_sch"
+			(at 147.32 83.1346 0)
+			(effects
+				(font
+					(size 1.27 1.27)
+				)
+				(justify left top)
+			)
+		)
+		(instances
+			(project "pillbus"
+				(path "/eae9d418-f407-4ce6-ae70-138b36f2a986"
+					(page "8")
+				)
+			)
+		)
+	)
+	(sheet
+		(at 196.85 121.92)
+		(size 74.93 8.89)
+		(fields_autoplaced yes)
+		(stroke
+			(width 0.1524)
+			(type solid)
+		)
+		(fill
+			(color 0 0 0 0.0000)
+		)
 		(property "Sheetname" "leds2"
 			(at 196.85 121.2084 0)
@@
 				)
 			)
+		)
+	)
+	(sheet
+		(at 21.59 21.59)
+		(size 43.18 59.69)
+		(fields_autoplaced yes)
+		(stroke
+			(width 0.1524)
+			(type solid)
+		)
+		(fill
+			(color 0 0 0 0.0000)
+		)
+		(property "Sheetname" "stm32pill"
+			(at 21.59 20.8784 0)
+			(effects
+				(font
+					(size 1.27 1.27)
+				)
+				(justify left bottom)
+			)
+		)
+		(property "Sheetfile" "stm32pill.kicad_sch"
+			(at 21.59 81.8646 0)
+			(effects
+				(font
+					(size 1.27 1.27)
+				)
+				(justify left top)
+			)
+		)
+		(instances
+			(project "pillbus"
+				(path "/eae9d418-f407-4ce6-ae70-138b36f2a986"
+					(page "6")
+				)
+			)
