File: hw/stm32-pillbus/pillbus.kicad_pcb (KiCad board)
At the start: 2 copper layers, 100 x 100 mm, 76 parts, among them J10 IDE, J11 IDE, J12 IDE, J13 IDE, J14 IDE, J15 IDE, J16 IDE, J17 IDE, J18 IDE, J9 IDE, U1 STM32F103C8T6, U2 STM32F103C8T6, U3 STM32F103C8T6, U4 STM32F103C8T6, U5 STM32F103C8T6

Commit message: stm32-panel
Parts:
- removed ? (x4): , 
- removed C16, C17, C18, C19, C20: CL21B103KBANNNC, jlcpcb:C0805
- removed IDE_STM, J10, J12, J14, J16, J18: IDE, ribbon:IDE STM AB
- removed J11, J13, J15, J17, J9: IDE, ribbon:IDE STM CD
- removed REF** (x4): PTH, base:PTH 1.7mm
- added 3.3V1: ~, base:PTH 1.7mm, F.Cu at (58.6, 64.8)
- added 3.3V2: ~, base:PTH 1.7mm, F.Cu at (81.3, 64.8)
- added 3.3V3: ~, base:PTH 1.7mm, F.Cu at (104.1, 64.8)
- added 3.3V4: ~, base:PTH 1.7mm, F.Cu at (127.0, 64.8)
- added 3.3V5: ~, base:PTH 1.7mm, F.Cu at (64.8, 96.5)
- added B1: ~, base:3x PTH 1.7mm, F.Cu at (43.3, 53.3)
- added B2: ~, base:3x PTH 1.7mm, F.Cu at (66.0, 53.3)
- added B3: ~, base:3x PTH 1.7mm, F.Cu at (88.9, 53.3)
- added B4: ~, base:3x PTH 1.7mm, F.Cu at (111.7, 53.4)
- added B5: ~, base:3x PTH 1.7mm, F.Cu at (53.3, 111.8)
- added CVcc1: 4.7uF, jlcpcb:C1206, F.Cu at (50.9, 58.4)
- added CVcc2: 4.7uF, jlcpcb:C1206, F.Cu at (73.7, 58.4)
- added CVcc3: 4.7uF, jlcpcb:C1206, F.Cu at (96.5, 58.4)
- added CVcc4: 4.7uF, jlcpcb:C1206, F.Cu at (119.4, 58.4)
- added CVcc5: 4.7uF, jlcpcb:C1206, F.Cu at (58.4, 104.1)
- added CVssA1: 1μF, jlcpcb:C0402, F.Cu at (47.7, 75.6)
- added CVssA2: 1μF, jlcpcb:C0402, F.Cu at (70.4, 75.6)
- added CVssA3: 1μF, jlcpcb:C0402, F.Cu at (93.3, 75.6)
- added CVssA4: 1μF, jlcpcb:C0402, F.Cu at (116.1, 75.6)
- added CVssA5: 1μF, jlcpcb:C0402, F.Cu at (75.6, 107.4)
- added CVssAn1: 10nF, jlcpcb:C0402, F.Cu at (47.5, 73.8)
- added CVssAn2: 10nF, jlcpcb:C0402, F.Cu at (70.3, 73.8)
- added CVssAn3: 10nF, jlcpcb:C0402, F.Cu at (93.1, 73.8)
- added CVssAn4: 10nF, jlcpcb:C0402, F.Cu at (116.0, 73.8)
- added CVssAn5: 10nF, jlcpcb:C0402, F.Cu at (73.8, 107.5)
- added Cosc1: 30pF, jlcpcb:C0402, F.Cu at (42.7, 74.1)
- added Cosc10: 30pF, jlcpcb:C0402, F.Cu at (75.6, 109.9)
- added Cosc2: 30pF, jlcpcb:C0402, F.Cu at (45.2, 75.6)
- added Cosc3: 30pF, jlcpcb:C0402, F.Cu at (65.4, 74.1)
- added Cosc4: 30pF, jlcpcb:C0402, F.Cu at (67.9, 75.6)
- added Cosc5: 30pF, jlcpcb:C0402, F.Cu at (88.3, 74.1)
- added Cosc6: 30pF, jlcpcb:C0402, F.Cu at (90.8, 75.6)
- added Cosc7: 30pF, jlcpcb:C0402, F.Cu at (111.1, 74.1)
- added Cosc8: 30pF, jlcpcb:C0402, F.Cu at (113.6, 75.6)
- added Cosc9: 30pF, jlcpcb:C0402, F.Cu at (74.1, 112.4)
- added Crst1: 100nF, jlcpcb:C0402, F.Cu at (54.2, 74.0)
- added Crst2: 100nF, jlcpcb:C0402, F.Cu at (77.0, 74.0)
- added Crst3: 100nF, jlcpcb:C0402, F.Cu at (99.8, 74.0)
- added Crst4: 100nF, jlcpcb:C0402, F.Cu at (122.7, 74.1)
- added Crst5: 100nF, jlcpcb:C0402, F.Cu at (74.0, 100.8)
- added DI1: ~, base:PTH 1.7mm, F.Cu at (56.0, 76.2)
- added DI2: ~, base:PTH 1.7mm, F.Cu at (78.7, 76.2)
- added DI3: ~, base:PTH 1.7mm, F.Cu at (101.6, 76.2)
- added DI4: ~, base:PTH 1.7mm, F.Cu at (124.4, 76.2)
- added DI5: ~, base:PTH 1.7mm, F.Cu at (76.2, 99.1)
- added GND1: ~, base:PTH 1.7mm, F.Cu at (58.6, 67.5)
- added GND2: ~, base:PTH 1.7mm, F.Cu at (81.3, 67.5)
- added GND3: ~, base:PTH 1.7mm, F.Cu at (104.1, 67.5)
- added GND4: ~, base:PTH 1.7mm, F.Cu at (127.0, 67.5)
- added GND5: ~, base:PTH 1.7mm, F.Cu at (67.5, 96.5)
- added IDE_STM_A1: ~, ribbon:IDE STM A, F.Cu at (60.8, 40.6)
- added IDE_STM_A2: ~, ribbon:IDE STM A, F.Cu at (83.6, 40.6)
- added IDE_STM_A3: ~, ribbon:IDE STM A, F.Cu at (106.4, 40.6)
- added IDE_STM_A4: ~, ribbon:IDE STM A, F.Cu at (129.3, 40.7)
- added IDE_STM_A5: ~, ribbon:IDE STM A, F.Cu at (40.6, 94.2)
- added IDE_STM_B1: ~, ribbon:IDE STM B, F.Cu at (61.1, 66.0)
- added IDE_STM_B2: ~, ribbon:IDE STM B, F.Cu at (83.8, 66.0)
- added IDE_STM_B3: ~, ribbon:IDE STM B, F.Cu at (106.7, 66.0)
- added IDE_STM_B4: ~, ribbon:IDE STM B, F.Cu at (129.5, 66.1)
- added IDE_STM_B5: ~, ribbon:IDE STM B, F.Cu at (66.0, 94.0)
- added IDE_STM_C1: ~, ribbon:IDE STM C, F.Cu at (40.8, 40.6)
- added IDE_STM_C2: ~, ribbon:IDE STM C, F.Cu at (63.5, 40.6)
- added IDE_STM_C3: ~, ribbon:IDE STM C, F.Cu at (86.4, 40.6)
- added IDE_STM_C4: ~, ribbon:IDE STM C, F.Cu at (109.2, 40.7)
- added IDE_STM_C5: ~, ribbon:IDE STM C, F.Cu at (40.6, 114.3)
- added IDE_STM_D1: ~, ribbon:IDE STM D, F.Cu at (40.8, 88.9)
- added IDE_STM_D2: ~, ribbon:IDE STM D, F.Cu at (63.5, 88.9)
- added IDE_STM_D3: ~, ribbon:IDE STM D, F.Cu at (86.4, 88.9)
- added IDE_STM_D4: ~, ribbon:IDE STM D, F.Cu at (109.2, 88.9)
- added IDE_STM_D5: ~, ribbon:IDE STM D, F.Cu at (88.9, 114.3)
- added JPLed1: SolderJumper_3_Open, Jumper:SolderJumper-3_P1.3mm_Open_RoundedPad1.0x1.5mm, B.Cu at (50.9, 41.9)
- added JPLed2: SolderJumper_3_Open, Jumper:SolderJumper-3_P1.3mm_Open_RoundedPad1.0x1.5mm, B.Cu at (73.7, 41.9)
- added JPLed3: SolderJumper_3_Open, Jumper:SolderJumper-3_P1.3mm_Open_RoundedPad1.0x1.5mm, B.Cu at (96.5, 41.9)
- added JPLed4: SolderJumper_3_Open, Jumper:SolderJumper-3_P1.3mm_Open_RoundedPad1.0x1.5mm, B.Cu at (119.4, 41.9)
- added JPLed5: SolderJumper_3_Open, Jumper:SolderJumper-3_P1.3mm_Open_RoundedPad1.0x1.5mm, B.Cu at (41.9, 104.1)
- added JPReset1: SolderJumper_2_Open, Jumper:SolderJumper-2_P1.3mm_Open_RoundedPad1.0x1.5mm, B.Cu at (50.9, 78.7)
- added JPReset2: SolderJumper_2_Open, Jumper:SolderJumper-2_P1.3mm_Open_RoundedPad1.0x1.5mm, B.Cu at (73.6, 78.7)
- added JPReset3: SolderJumper_2_Open, Jumper:SolderJumper-2_P1.3mm_Open_RoundedPad1.0x1.5mm, B.Cu at (96.4, 78.7)
- added JPReset4: SolderJumper_2_Open, Jumper:SolderJumper-2_P1.3mm_Open_RoundedPad1.0x1.5mm, B.Cu at (119.3, 78.8)
- added JPReset5: SolderJumper_2_Open, Jumper:SolderJumper-2_P1.3mm_Open_RoundedPad1.0x1.5mm, B.Cu at (78.7, 104.2)
- added JPRscl1: SolderJumper_2_Open, Jumper:SolderJumper-2_P1.3mm_Open_RoundedPad1.0x1.5mm, B.Cu at (44.6, 58.4)
- added JPRscl2: SolderJumper_2_Open, Jumper:SolderJumper-2_P1.3mm_Open_RoundedPad1.0x1.5mm, B.Cu at (67.3, 58.4)
- added JPRscl3: SolderJumper_2_Open, Jumper:SolderJumper-2_P1.3mm_Open_RoundedPad1.0x1.5mm, B.Cu at (90.2, 58.4)
- added JPRscl4: SolderJumper_2_Open, Jumper:SolderJumper-2_P1.3mm_Open_RoundedPad1.0x1.5mm, B.Cu at (113.0, 58.4)
- added JPRscl5: SolderJumper_2_Open, Jumper:SolderJumper-2_P1.3mm_Open_RoundedPad1.0x1.5mm, B.Cu at (58.4, 110.5)
- added JPRsda1: SolderJumper_2_Open, Jumper:SolderJumper-2_P1.3mm_Open_RoundedPad1.0x1.5mm, B.Cu at (44.6, 61.0)
- added JPRsda2: SolderJumper_2_Open, Jumper:SolderJumper-2_P1.3mm_Open_RoundedPad1.0x1.5mm, B.Cu at (67.3, 61.0)
- added JPRsda3: SolderJumper_2_Open, Jumper:SolderJumper-2_P1.3mm_Open_RoundedPad1.0x1.5mm, B.Cu at (90.2, 61.0)
- added JPRsda4: SolderJumper_2_Open, Jumper:SolderJumper-2_P1.3mm_Open_RoundedPad1.0x1.5mm, B.Cu at (113.0, 61.0)
- added JPRsda5: SolderJumper_2_Open, Jumper:SolderJumper-2_P1.3mm_Open_RoundedPad1.0x1.5mm, B.Cu at (61.0, 110.5)
- added JPV1: SolderJumper_2_Open, Jumper:SolderJumper-2_P1.3mm_Open_RoundedPad1.0x1.5mm, B.Cu at (44.0, 40.6)
- added JPV2: SolderJumper_2_Open, Jumper:SolderJumper-2_P1.3mm_Open_RoundedPad1.0x1.5mm, B.Cu at (66.7, 40.6)
- added JPV3: SolderJumper_2_Open, Jumper:SolderJumper-2_P1.3mm_Open_RoundedPad1.0x1.5mm, B.Cu at (89.5, 40.6)
- added JPV4: SolderJumper_2_Open, Jumper:SolderJumper-2_P1.3mm_Open_RoundedPad1.0x1.5mm, B.Cu at (112.4, 40.7)
- added JPV5: SolderJumper_2_Open, Jumper:SolderJumper-2_P1.3mm_Open_RoundedPad1.0x1.5mm, B.Cu at (40.6, 111.1)
- added JPdn1: SolderJumper_2_Open, Jumper:SolderJumper-2_P1.3mm_Open_RoundedPad1.0x1.5mm, B.Cu at (58.2, 43.2)
- added JPdn2: SolderJumper_2_Open, Jumper:SolderJumper-2_P1.3mm_Open_RoundedPad1.0x1.5mm, B.Cu at (80.9, 43.2)
- added JPdn3: SolderJumper_2_Open, Jumper:SolderJumper-2_P1.3mm_Open_RoundedPad1.0x1.5mm, B.Cu at (103.7, 43.2)
- added JPdn4: SolderJumper_2_Open, Jumper:SolderJumper-2_P1.3mm_Open_RoundedPad1.0x1.5mm, B.Cu at (126.6, 43.2)
- added JPdn5: SolderJumper_2_Open, Jumper:SolderJumper-2_P1.3mm_Open_RoundedPad1.0x1.5mm, B.Cu at (43.2, 96.9)
- added JPdp1: SolderJumper_2_Open, Jumper:SolderJumper-2_P1.3mm_Open_RoundedPad1.0x1.5mm, B.Cu at (44.0, 45.7)
- added JPdp2: SolderJumper_2_Open, Jumper:SolderJumper-2_P1.3mm_Open_RoundedPad1.0x1.5mm, B.Cu at (66.7, 45.7)
- added JPdp3: SolderJumper_2_Open, Jumper:SolderJumper-2_P1.3mm_Open_RoundedPad1.0x1.5mm, B.Cu at (89.5, 45.7)
- added JPdp4: SolderJumper_2_Open, Jumper:SolderJumper-2_P1.3mm_Open_RoundedPad1.0x1.5mm, B.Cu at (112.4, 45.7)
- added JPdp5: SolderJumper_2_Open, Jumper:SolderJumper-2_P1.3mm_Open_RoundedPad1.0x1.5mm, B.Cu at (45.7, 111.1)
- added JPpuUSB1: SolderJumper_3_Open, Jumper:SolderJumper-3_P1.3mm_Open_RoundedPad1.0x1.5mm, B.Cu at (52.1, 47.1)
- added JPpuUSB2: SolderJumper_3_Open, Jumper:SolderJumper-3_P1.3mm_Open_RoundedPad1.0x1.5mm, B.Cu at (74.8, 47.1)
- added JPpuUSB3: SolderJumper_3_Open, Jumper:SolderJumper-3_P1.3mm_Open_RoundedPad1.0x1.5mm, B.Cu at (97.7, 47.1)
- added JPpuUSB4: SolderJumper_3_Open, Jumper:SolderJumper-3_P1.3mm_Open_RoundedPad1.0x1.5mm, B.Cu at (120.5, 47.1)
- added JPpuUSB5: SolderJumper_3_Open, Jumper:SolderJumper-3_P1.3mm_Open_RoundedPad1.0x1.5mm, B.Cu at (47.1, 103.0)
- added JPpuUSBconst1: SolderJumper_2_Open, Jumper:SolderJumper-2_P1.3mm_Open_RoundedPad1.0x1.5mm, B.Cu at (52.1, 52.5)
- added JPpuUSBconst2: SolderJumper_2_Open, Jumper:SolderJumper-2_P1.3mm_Open_RoundedPad1.0x1.5mm, B.Cu at (74.9, 52.5)
- added JPpuUSBconst3: SolderJumper_2_Open, Jumper:SolderJumper-2_P1.3mm_Open_RoundedPad1.0x1.5mm, B.Cu at (97.7, 52.5)
- added JPpuUSBconst4: SolderJumper_2_Open, Jumper:SolderJumper-2_P1.3mm_Open_RoundedPad1.0x1.5mm, B.Cu at (120.5, 52.5)
- added JPpuUSBconst5: SolderJumper_2_Open, Jumper:SolderJumper-2_P1.3mm_Open_RoundedPad1.0x1.5mm, B.Cu at (52.5, 102.9)
- added JPvbus1: SolderJumper_2_Open, Jumper:SolderJumper-2_P1.3mm_Open_RoundedPad1.0x1.5mm, B.Cu at (44.0, 43.2)
- added JPvbus2: SolderJumper_2_Open, Jumper:SolderJumper-2_P1.3mm_Open_RoundedPad1.0x1.5mm, B.Cu at (66.7, 43.2)
- added JPvbus3: SolderJumper_2_Open, Jumper:SolderJumper-2_P1.3mm_Open_RoundedPad1.0x1.5mm, B.Cu at (89.5, 43.2)
- added JPvbus4: SolderJumper_2_Open, Jumper:SolderJumper-2_P1.3mm_Open_RoundedPad1.0x1.5mm, B.Cu at (112.4, 43.2)
- added JPvbus5: SolderJumper_2_Open, Jumper:SolderJumper-2_P1.3mm_Open_RoundedPad1.0x1.5mm, B.Cu at (43.2, 111.1)
- added JSH1: ~, base:PTH 1.7mm, F.Cu at (50.9, 81.3)
- added JSH2: ~, base:PTH 1.7mm, F.Cu at (73.7, 81.3)
- added JSH3: ~, base:PTH 1.7mm, F.Cu at (96.5, 81.3)
- added JSH4: ~, base:PTH 1.7mm, F.Cu at (119.4, 81.3)
- added JSH5: ~, base:PTH 1.7mm, F.Cu at (81.3, 104.1)
- added JSL1: ~, base:PTH 1.7mm, F.Cu at (45.9, 81.3)
- added JSL2: ~, base:PTH 1.7mm, F.Cu at (68.6, 81.3)
- added JSL3: ~, base:PTH 1.7mm, F.Cu at (91.4, 81.3)
- added JSL4: ~, base:PTH 1.7mm, F.Cu at (114.3, 81.3)
- added JSL5: ~, base:PTH 1.7mm, F.Cu at (81.3, 109.2)
- added JVbat1: VBAT, TestPoint:TestPoint_THTPad_D1.0mm_Drill0.5mm, F.Cu at (43.3, 77.5)
- added JVbat2: VBAT, TestPoint:TestPoint_THTPad_D1.0mm_Drill0.5mm, F.Cu at (66.0, 77.5)
- added JVbat3: VBAT, TestPoint:TestPoint_THTPad_D1.0mm_Drill0.5mm, F.Cu at (88.9, 77.5)
- added JVbat4: VBAT, TestPoint:TestPoint_THTPad_D1.0mm_Drill0.5mm, F.Cu at (111.7, 77.5)
- added JVbat5: VBAT, TestPoint:TestPoint_THTPad_D1.0mm_Drill0.5mm, F.Cu at (77.5, 111.8)
- added Jled1: ~, base:PTH 1.7mm, F.Cu at (58.6, 50.8)
- added Jled2: ~, base:PTH 1.7mm, F.Cu at (81.3, 50.8)
- added Jled3: ~, base:PTH 1.7mm, F.Cu at (104.1, 50.8)
- added Jled4: ~, base:PTH 1.7mm, F.Cu at (127.0, 50.8)
- added Jled5: ~, base:PTH 1.7mm, F.Cu at (50.8, 96.5)
- added JpuUSB1: ~, base:PTH 1.7mm, F.Cu at (56.0, 50.8)
- added JpuUSB2: ~, base:PTH 1.7mm, F.Cu at (78.7, 50.8)
- added JpuUSB3: ~, base:PTH 1.7mm, F.Cu at (101.6, 50.8)
- added JpuUSB4: ~, base:PTH 1.7mm, F.Cu at (124.4, 50.8)
- added JpuUSB5: ~, base:PTH 1.7mm, F.Cu at (50.8, 99.1)
- added Jrst1: ~, base:PTH 1.7mm, F.Cu at (48.4, 81.3)
- added Jrst2: ~, base:PTH 1.7mm, F.Cu at (71.1, 81.3)
- added Jrst3: ~, base:PTH 1.7mm, F.Cu at (94.0, 81.3)
- added Jrst4: ~, base:PTH 1.7mm, F.Cu at (116.8, 81.3)
- added Jrst5: ~, base:PTH 1.7mm, F.Cu at (81.3, 106.7)
- added L1: 100Ω@100MHz, jlcpcb:L0805, F.Cu at (48.0, 49.6)
- added L2: 100Ω@100MHz, jlcpcb:L0805, F.Cu at (70.8, 49.6)
- added L3: 100Ω@100MHz, jlcpcb:L0805, F.Cu at (93.6, 49.6)
- added L4: 100Ω@100MHz, jlcpcb:L0805, F.Cu at (116.5, 49.7)
- added L5: 100Ω@100MHz, jlcpcb:L0805, F.Cu at (49.6, 107.0)
- added LED33: Green, jlcpcb:LED0805-R-RD, F.Cu at (58.1, 47.4)
- added LED34: Green, jlcpcb:LED0805-R-RD, F.Cu at (80.8, 47.4)
- added LED35: Green, jlcpcb:LED0805-R-RD, F.Cu at (103.6, 47.4)
- added LED36: Green, jlcpcb:LED0805-R-RD, F.Cu at (126.5, 47.4)
- added LED37: Green, jlcpcb:LED0805-R-RD, F.Cu at (47.4, 97.0)
- added LVssA1: 18nH, jlcpcb:L0201, F.Cu at (48.2, 76.7)
- added LVssA2: 18nH, jlcpcb:L0201, F.Cu at (70.9, 76.7)
- added LVssA3: 18nH, jlcpcb:L0201, F.Cu at (93.8, 76.7)
- added LVssA4: 18nH, jlcpcb:L0201, F.Cu at (116.6, 76.7)
- added LVssA5: 18nH, jlcpcb:L0201, F.Cu at (76.7, 106.9)
- added RGB1: LED WS2812B-S XL-5050RGBC, jlcpcb:LED-SMD_4P-L5.0-W5.0-TL-1, F.Cu at (56.1, 79.8)
- added RGB2: LED WS2812B-S XL-5050RGBC, jlcpcb:LED-SMD_4P-L5.0-W5.0-TL-1, F.Cu at (78.8, 79.8)
- added RGB3: LED WS2812B-S XL-5050RGBC, jlcpcb:LED-SMD_4P-L5.0-W5.0-TL-1, F.Cu at (101.7, 79.8)
- added RGB4: LED WS2812B-S XL-5050RGBC, jlcpcb:LED-SMD_4P-L5.0-W5.0-TL-1, F.Cu at (124.5, 79.9)
- added RGB5: LED WS2812B-S XL-5050RGBC, jlcpcb:LED-SMD_4P-L5.0-W5.0-TL-1, F.Cu at (79.8, 99.0)
- added RVbusI1: 33kΩ, jlcpcb:R0402, F.Cu at (44.2, 44.5)
- added RVbusI2: 33kΩ, jlcpcb:R0402, F.Cu at (66.9, 44.5)
- added RVbusI3: 33kΩ, jlcpcb:R0402, F.Cu at (89.7, 44.5)
- added RVbusI4: 33kΩ, jlcpcb:R0402, F.Cu at (112.6, 44.5)
- added RVbusI5: 33kΩ, jlcpcb:R0402, F.Cu at (44.5, 110.9)
- added RVbusO1: 82kΩ, jlcpcb:R0402, F.Cu at (44.2, 43.2)
- added RVbusO2: 82kΩ, jlcpcb:R0402, F.Cu at (66.9, 43.2)
- added RVbusO3: 82kΩ, jlcpcb:R0402, F.Cu at (89.7, 43.2)
- added RVbusO4: 82kΩ, jlcpcb:R0402, F.Cu at (112.6, 43.2)
- added RVbusO5: 82kΩ, jlcpcb:R0402, F.Cu at (43.2, 110.9)
- added Rled1: 1k-1.5k, jlcpcb:R0402, F.Cu at (55.8, 48.9)
- added Rled2: 1k-1.5k, jlcpcb:R0402, F.Cu at (78.5, 48.9)
- added Rled3: 1k-1.5k, jlcpcb:R0402, F.Cu at (101.3, 48.9)
- added Rled4: 1k-1.5k, jlcpcb:R0402, F.Cu at (124.2, 48.9)
- added Rled5: 1k-1.5k, jlcpcb:R0402, F.Cu at (48.9, 99.3)
- added Rpd1: 10kΩ, jlcpcb:R0402, F.Cu at (57.9, 83.8)
- added Rpd2: 10kΩ, jlcpcb:R0402, F.Cu at (80.6, 83.8)
- added Rpd3: 10kΩ, jlcpcb:R0402, F.Cu at (103.5, 83.8)
- added Rpd4: 10kΩ, jlcpcb:R0402, F.Cu at (126.3, 83.8)
- added Rpd5: 10kΩ, jlcpcb:R0402, F.Cu at (83.8, 97.2)
- added Rpu1: 10kΩ, jlcpcb:R0402, F.Cu at (43.7, 83.8)
- added Rpu2: 10kΩ, jlcpcb:R0402, F.Cu at (66.4, 83.8)
- added Rpu3: 10kΩ, jlcpcb:R0402, F.Cu at (89.2, 83.8)
- added Rpu4: 10kΩ, jlcpcb:R0402, F.Cu at (112.1, 83.8)
- added Rpu5: 10kΩ, jlcpcb:R0402, F.Cu at (83.8, 111.4)
- added RpuUSB1: 1.5kΩ, jlcpcb:R0402, F.Cu at (53.9, 49.1)
- added RpuUSB2: 1.5kΩ, jlcpcb:R0402, F.Cu at (76.7, 49.1)
- added RpuUSB3: 1.5kΩ, jlcpcb:R0402, F.Cu at (99.5, 49.1)
- added RpuUSB4: 1.5kΩ, jlcpcb:R0402, F.Cu at (122.4, 49.1)
- added RpuUSB5: 1.5kΩ, jlcpcb:R0402, F.Cu at (49.1, 101.1)
- added Rscl1: 2.2kΩ, jlcpcb:R0402, F.Cu at (43.0, 67.0)
- added Rscl2: 2.2kΩ, jlcpcb:R0402, F.Cu at (65.7, 67.0)
- added Rscl3: 2.2kΩ, jlcpcb:R0402, F.Cu at (88.6, 67.0)
- added Rscl4: 2.2kΩ, jlcpcb:R0402, F.Cu at (111.4, 67.0)
- added Rscl5: 2.2kΩ, jlcpcb:R0402, F.Cu at (67.0, 112.1)
- added Rsda1: 2.2kΩ, jlcpcb:R0402, F.Cu at (44.3, 67.0)
- added Rsda2: 2.2kΩ, jlcpcb:R0402, F.Cu at (67.1, 67.0)
- added Rsda3: 2.2kΩ, jlcpcb:R0402, F.Cu at (89.9, 67.0)
- added Rsda4: 2.2kΩ, jlcpcb:R0402, F.Cu at (112.8, 67.0)
- added Rsda5: 2.2kΩ, jlcpcb:R0402, F.Cu at (67.0, 110.7)
- added SW1: Tactile Switch, jlcpcb:SW-SMD_4P-L5.1-W5.1-P3.70-LS6.5-TL_H1.5, F.Cu at (46.5, 86.9)
- added SW10: Tactile Switch, jlcpcb:SW-SMD_4P-L5.1-W5.1-P3.70-LS6.5-TL_H1.5, F.Cu at (86.9, 99.9)
- added SW2: Tactile Switch, jlcpcb:SW-SMD_4P-L5.1-W5.1-P3.70-LS6.5-TL_H1.5, F.Cu at (55.2, 86.9)
- added SW3: Tactile Switch, jlcpcb:SW-SMD_4P-L5.1-W5.1-P3.70-LS6.5-TL_H1.5, F.Cu at (69.2, 86.9)
- added SW4: Tactile Switch, jlcpcb:SW-SMD_4P-L5.1-W5.1-P3.70-LS6.5-TL_H1.5, F.Cu at (77.9, 86.9)
- added SW5: Tactile Switch, jlcpcb:SW-SMD_4P-L5.1-W5.1-P3.70-LS6.5-TL_H1.5, F.Cu at (92.1, 86.9)
- added SW6: Tactile Switch, jlcpcb:SW-SMD_4P-L5.1-W5.1-P3.70-LS6.5-TL_H1.5, F.Cu at (100.8, 86.9)
- added SW7: Tactile Switch, jlcpcb:SW-SMD_4P-L5.1-W5.1-P3.70-LS6.5-TL_H1.5, F.Cu at (114.9, 87.0)
- added SW8: Tactile Switch, jlcpcb:SW-SMD_4P-L5.1-W5.1-P3.70-LS6.5-TL_H1.5, F.Cu at (123.6, 87.0)
- added SW9: Tactile Switch, jlcpcb:SW-SMD_4P-L5.1-W5.1-P3.70-LS6.5-TL_H1.5, F.Cu at (86.9, 108.6)
- added U10: STM32F103C8T6, jlcpcb:LQFP-48_L7.0-W7.0-P0.50-LS9.0-BL, F.Cu at (67.3, 104.1)
- added U6: STM32F103C8T6, jlcpcb:LQFP-48_L7.0-W7.0-P0.50-LS9.0-BL, F.Cu at (96.5, 67.3)
- added U7: 3.3V Voltage Regulator 200mA, jlcpcb:SOT-23-3_L2.9-W1.6-P1.90-LS2.8-BR, F.Cu at (112.4, 48.9)
- added U8: STM32F103C8T6, jlcpcb:LQFP-48_L7.0-W7.0-P0.50-LS9.0-BL, F.Cu at (119.4, 67.3)
- added U9: 3.3V Voltage Regulator 200mA, jlcpcb:SOT-23-3_L2.9-W1.6-P1.90-LS2.8-BR, F.Cu at (48.9, 111.1)
- added USB1: USB_C, jlcpcb:USB-C_SMD-TYPE-C-31-M-12, F.Cu at (51.0, 44.6)
- added USB2: USB_C, jlcpcb:USB-C_SMD-TYPE-C-31-M-12, F.Cu at (73.7, 44.6)
- added USB3: USB_C, jlcpcb:USB-C_SMD-TYPE-C-31-M-12, F.Cu at (96.5, 44.6)
- added USB4: USB_C, jlcpcb:USB-C_SMD-TYPE-C-31-M-12, F.Cu at (119.4, 44.6)
- added USB5: USB_C, jlcpcb:USB-C_SMD-TYPE-C-31-M-12, F.Cu at (44.6, 104.1)
- added VSSA1: VSSA, TestPoint:TestPoint_THTPad_D1.0mm_Drill0.5mm, F.Cu at (45.9, 77.5)
- added VSSA2: VSSA, TestPoint:TestPoint_THTPad_D1.0mm_Drill0.5mm, F.Cu at (68.6, 77.5)
- added VSSA3: VSSA, TestPoint:TestPoint_THTPad_D1.0mm_Drill0.5mm, F.Cu at (91.4, 77.5)
- added VSSA4: VSSA, TestPoint:TestPoint_THTPad_D1.0mm_Drill0.5mm, F.Cu at (114.3, 77.5)
- added VSSA5: VSSA, TestPoint:TestPoint_THTPad_D1.0mm_Drill0.5mm, F.Cu at (77.5, 109.2)
- added X1: Crystal 12MHz X322512MSB4SI, jlcpcb:CRYSTAL-SMD_4P-L3.2-W2.5-BL, F.Cu at (45.1, 72.9)
- added X2: Crystal 12MHz X322512MSB4SI, jlcpcb:CRYSTAL-SMD_4P-L3.2-W2.5-BL, F.Cu at (67.8, 72.9)
- added X3: Crystal 12MHz X322512MSB4SI, jlcpcb:CRYSTAL-SMD_4P-L3.2-W2.5-BL, F.Cu at (90.6, 72.9)
- added X4: Crystal 12MHz X322512MSB4SI, jlcpcb:CRYSTAL-SMD_4P-L3.2-W2.5-BL, F.Cu at (113.5, 72.9)
- added X5: Crystal 12MHz X322512MSB4SI, jlcpcb:CRYSTAL-SMD_4P-L3.2-W2.5-BL, F.Cu at (72.9, 110.0)
- C1, C10, C11, C12, C13, C14, C15, C2, C3, C4, C5, C6, C7, C8, C9: value CL21B103KBANNNC -> 100nF; footprint jlcpcb:C0805 -> jlcpcb:C0402
- U1, U3, U5: value STM32F103C8T6 -> 3.3V Voltage Regulator 200mA; footprint jlcpcb:LQFP-48_L7.0-W7.0-P0.50-LS9.0-BL -> jlcpcb:SOT-23-3_L2.9-W1.6-P1.90-LS2.8-BR
- moved U1 60.1 mm to (44.0, 48.9), turned to 0 degrees
- moved U3 55.4 mm to (66.7, 48.9), turned to 0 degrees
- moved C15 52.2 mm to (65.1, 110.6), turned to 90 degrees
- moved C2 51.7 mm to (53.2, 60.9), turned to -90 degrees
- moved C3 41.3 mm to (44.5, 65.1), turned to 0 degrees
- moved C14 40.5 mm to (60.9, 101.9), turned to 0 degrees
- moved C1 39.7 mm to (57.4, 69.5), turned to 180 degrees
- moved C13 31.2 mm to (69.5, 97.7), turned to -90 degrees
- moved C4 30.6 mm to (80.1, 69.5), turned to 180 degrees
- moved C7 30.0 mm to (103.0, 69.5), turned to 180 degrees
- moved C9 29.2 mm to (90.1, 65.1), turned to 0 degrees
- moved U4 23.1 mm to (73.7, 67.3), turned to -45 degrees
- moved U2 22.5 mm to (50.9, 67.3), turned to -45 degrees
- moved C8 19.8 mm to (98.8, 60.9), turned to -90 degrees
- moved U5 19.2 mm to (89.6, 48.9), turned to 0 degrees
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Connections:
- U1 pad 1: /stm32pill/VBAT -> GND
- U1 pad 2: Net-(J10-IDE40_STM2) -> /stm32pill/VBUS
- U1 pad 3: Net-(J10-IDE38_STM3) -> +3.3V
- U2 pad 1: /stm32pill1/VBAT -> /stm32pill/VBAT
- U2 pad 15: Net-(J12-IDE18_STM15) -> /stm32pill/SPI1 SCK
- U2 pad 16: Net-(J12-IDE16_STM16) -> /stm32pill/SPI1 MISO
- U2 pad 17: Net-(J12-IDE14_STM17) -> /stm32pill/SPI1 MOSI
- U2 pad 21: Net-(J12-IDE6_STM21) -> /stm32pill/I2C2 SCL, USART3 TX
- U2 pad 22: Net-(J12-IDE4_STM22) -> /stm32pill/I2C2 SDA, USART3 RX
- U2 pad 25: Net-(J11-IDE5_STM25) -> /stm32pill/SPI2 NSS
- U2 pad 26: Net-(J11-IDE7_STM26) -> /stm32pill/SPI2 SCK
- U2 pad 27: Net-(J11-IDE9_STM27) -> /stm32pill/SPI2 MISO
- U2 pad 28: Net-(J11-IDE11_STM28) -> /stm32pill/SPI2 MOSI
- U2 pad 30: Net-(J11-IDE15_STM30) -> /stm32pill/USART1 TX
- U2 pad 31: Net-(J11-IDE17_STM31) -> /stm32pill/USART1 RX
- U2 pad 32: Net-(J11-IDE19_STM32) -> /stm32pill/USBd-
- U2 pad 33: Net-(J11-IDE21_STM33) -> /stm32pill/USBd+
- U2 pad 43: Net-(J11-IDE3_STM43) -> /stm32pill/USB VBusSense
- U2 pad 44: /stm32pill1/Boot0 -> /stm32pill/Boot0
- U2 pad 45: Net-(J11-IDE37_STM45) -> /stm32pill/I2C1 SCL
- U2 pad 46: Net-(J11-IDE39_STM46) -> /stm32pill/I2C1 SDA
- U2 pad 5: /stm32pill1/OSC_IN -> /stm32pill/OSC_IN
- U2 pad 6: /stm32pill1/OSC_OUT -> /stm32pill/OSC_OUT
- U2 pad 7: /stm32pill1/NRST -> /stm32pill/NRST
- U2 pad 8: +3.3V -> /stm32pill/VSSA
- U3 pad 1: /stm32pill2/VBAT -> GND
- U3 pad 2: Net-(J14-IDE40_STM2) -> /stm32pill1/VBUS
- U3 pad 3: Net-(J14-IDE38_STM3) -> +3.3V
- U4 pad 1: /stm32pill3/VBAT -> /stm32pill1/VBAT
- U4 pad 15: Net-(J16-IDE18_STM15) -> /stm32pill1/SPI1 SCK
- U4 pad 16: Net-(J16-IDE16_STM16) -> /stm32pill1/SPI1 MISO
- U4 pad 17: Net-(J16-IDE14_STM17) -> /stm32pill1/SPI1 MOSI
- U4 pad 21: Net-(J16-IDE6_STM21) -> /stm32pill1/I2C2 SCL, USART3 TX
- U4 pad 22: Net-(J16-IDE4_STM22) -> /stm32pill1/I2C2 SDA, USART3 RX
- U4 pad 25: Net-(J15-IDE5_STM25) -> /stm32pill1/SPI2 NSS
- U4 pad 26: Net-(J15-IDE7_STM26) -> /stm32pill1/SPI2 SCK
- U4 pad 27: Net-(J15-IDE9_STM27) -> /stm32pill1/SPI2 MISO
- U4 pad 28: Net-(J15-IDE11_STM28) -> /stm32pill1/SPI2 MOSI
- U4 pad 30: Net-(J15-IDE15_STM30) -> /stm32pill1/USART1 TX
- U4 pad 31: Net-(J15-IDE17_STM31) -> /stm32pill1/USART1 RX
- U4 pad 32: Net-(J15-IDE19_STM32) -> /stm32pill1/USBd-
- U4 pad 33: Net-(J15-IDE21_STM33) -> /stm32pill1/USBd+
- U4 pad 43: Net-(J15-IDE3_STM43) -> /stm32pill1/USB VBusSense
- U4 pad 44: /stm32pill3/Boot0 -> /stm32pill1/Boot0
- U4 pad 45: Net-(J15-IDE37_STM45) -> /stm32pill1/I2C1 SCL
- U4 pad 46: Net-(J15-IDE39_STM46) -> /stm32pill1/I2C1 SDA
- U4 pad 5: /stm32pill3/OSC_IN -> /stm32pill1/OSC_IN
- U4 pad 6: /stm32pill3/OSC_OUT -> /stm32pill1/OSC_OUT
- U4 pad 7: /stm32pill3/NRST -> /stm32pill1/NRST
- U4 pad 8: +3.3V -> /stm32pill1/VSSA
- U5 pad 1: /stm32pill4/VBAT -> GND
- U5 pad 2: Net-(J18-IDE40_STM2) -> /stm32pill2/VBUS
- U5 pad 3: Net-(J18-IDE38_STM3) -> +3.3V
Routing:
- net /stm32pill2/USBd+: track 0.00 -> 3338.1 mm, vias 0 -> 3
- net /stm32pill4/USBd+: track 0.00 -> 3136.1 mm, vias 0 -> 3
- net /stm32pill3/USBd+: track 0.00 -> 3052.2 mm, vias 0 -> 3
- net /stm32pill/USBd+: track 0.00 -> 2521.6 mm, vias 0 -> 3
- net /stm32pill1/USBd+: track 0.00 -> 2416.1 mm, vias 0 -> 3
- net GND: track 344.5 -> 979.2 mm, vias 10 -> 110
- net +3.3V: track 667.9 -> 822.5 mm, vias 10 -> 35
- net /stm32pill2/USB VBusSense: track 0.00 -> 44.8 mm, vias 0 -> 1
- net /stm32pill1/USB VBusSense: track 0.00 -> 44.8 mm, vias 0 -> 1
- net /stm32pill3/USB VBusSense: track 0.00 -> 44.8 mm, vias 0 -> 1
- net /stm32pill/USB VBusSense: track 0.00 -> 44.8 mm, vias 0 -> 1
- net /stm32pill4/USB VBusSense: track 0.00 -> 44.8 mm, vias 0 -> 1
- net Net-(J9-IDE3_STM43): track 32.4 -> 0.00 mm, vias 2 -> 0
- net Net-(J15-IDE3_STM43): track 32.4 -> 0.00 mm, vias 2 -> 0
- net Net-(J13-IDE3_STM43): track 32.4 -> 0.00 mm, vias 2 -> 0
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- added copper zone on B.Cu, net GND
Other:
- board text added: "A"
- board text added: "B"
- board text added: "C"
- board text added: "D"
- board text added: "SCL"
- board text added: "SDA"

Commit message: bus
Parts:
- added RpuBoot1: 51kΩ, jlcpcb:R0402, F.Cu at (47.0, 54.8)
- added RpuBoot2: 51kΩ, jlcpcb:R0402, F.Cu at (69.9, 54.8)
- added RpuBoot3: 51kΩ, jlcpcb:R0402, F.Cu at (92.8, 54.8)
- added RpuBoot4: 51kΩ, jlcpcb:R0402, F.Cu at (115.6, 54.8)
- added RpuBoot5: 51kΩ, jlcpcb:R0402, F.Cu at (54.8, 107.9)
- IDE_STM_B1, IDE_STM_B2, IDE_STM_B3, IDE_STM_B4, IDE_STM_B5: footprint ribbon:IDE STM B -> ribbon:IDE STM B cut
- IDE_STM_D1, IDE_STM_D2, IDE_STM_D3, IDE_STM_D4, IDE_STM_D5: footprint ribbon:IDE STM D -> ribbon:IDE STM D cut
- LVssA1, LVssA2, LVssA3, LVssA4, LVssA5: value 18nH -> 15-30nH; footprint jlcpcb:L0201 -> jlcpcb:L0402
- RVbusI1, RVbusI2, RVbusI3, RVbusI4, RVbusI5: value 33kΩ -> 51kΩ
- RVbusO1, RVbusO2, RVbusO3, RVbusO4, RVbusO5: value 82kΩ -> 100kΩ
- moved IDE_STM_D1 22.0 mm to (40.6, 66.9), turned to 0 degrees
- moved IDE_STM_D2 22.0 mm to (63.5, 66.9), turned to 0 degrees
- moved IDE_STM_D3 22.0 mm to (86.4, 66.9), turned to 0 degrees
- moved IDE_STM_D5 22.0 mm to (66.9, 114.3), turned to 90 degrees
- moved IDE_STM_D4 22.0 mm to (109.2, 66.9), turned to 0 degrees
- moved DI1 10.3 mm to (50.8, 85.1)
- moved DI2 10.2 mm to (73.7, 85.1)
- moved DI3 10.2 mm to (96.5, 85.1)
- moved DI4 10.2 mm to (119.4, 85.1)
- moved DI5 10.2 mm to (85.1, 104.1)
- moved Rpd1 2.68 mm to (55.9, 82.0)
- moved Rpd4 2.58 mm to (124.4, 82.1)
- moved Rpd2 2.58 mm to (78.7, 82.0)
- moved Rpd3 2.58 mm to (101.6, 82.0)
- moved Rpd5 2.58 mm to (82.0, 99.1)
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Routing:
- net /stm32pill/USBd+: track 2521.6 -> 58.0 mm
- net /stm32pill2/USBd+: track 3338.1 -> 1043.5 mm
- net /stm32pill4/USBd+: track 3136.1 -> 1140.4 mm
- net /stm32pill1/USBd+: track 2416.1 -> 694.7 mm
- net /stm32pill3/USBd+: track 3052.2 -> 1400.9 mm
- net (no net): track 0.00 -> 366.6 mm, vias 0 -> 4
- net /stm32pill/USBd-: track 31.7 -> 0.00 mm, vias 2 -> 0
- net GND: track 979.2 -> 998.4 mm
- net Net-(DI1-Pin_1): track 2.02 -> 11.6 mm, vias 0 -> 2
- net Net-(DI5-Pin_1): track 2.02 -> 11.6 mm, vias 0 -> 2
- net Net-(DI3-Pin_1): track 2.02 -> 11.6 mm, vias 0 -> 2
- net Net-(DI2-Pin_1): track 2.02 -> 11.6 mm, vias 0 -> 2
- net Net-(DI4-Pin_1): track 2.02 -> 11.6 mm, vias 0 -> 2
- net /stm32pill/VBUS: track 8.36 -> 0.00 mm, vias 2 -> 0
- net /stm32pill2/USB VBusSense: track 44.8 -> 37.3 mm, vias 1 -> 2
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Other:
- outline, holes or cut-outs redrawn
- board text added: "Flash UART"
- board text added: "TX RX"
- board text added: "https://github.com/johannesloetzsch/pillbus"
