File: hw/kicad-hierpcb/stm32pill.kicad_pcb (KiCad board)
At the start: 2 copper layers, 23.8 x 49 mm, 63 parts, among them SW1 Tactile Switch, SW2 Tactile Switch, U1 3.3V Voltage Regulator 200mA, X1 Crystal 12MHz X322512MSB4SI

Commit message: boot0: pullDown + serial resistor
Parts:
- added RSBoot1: 51kΩ, jlcpcb:R0402, F.Cu at (29.0, 40.8)
- turned RpuBoot1 to 180 degrees
Connections:
- MCU1 pad 44: /Boot0 -> Net-(MCU1-BOOT0)
- RpuBoot1 pad 1: +3.3V -> /Boot0
- RpuBoot1 pad 2: /Boot0 -> GND
Routing:
- net /Boot0: track 19.8 -> 7.43 mm, vias 3 -> 1
- net Net-(MCU1-BOOT0): track 0.00 -> 12.2 mm, vias 0 -> 2
- net GND: track 48.1 -> 49.7 mm, vias 20 -> 21
- net +3.3V: track 112.1 -> 111.2 mm
Other:
- board text added: "SWCLK"
- board text added: "SWDIO"
